File: main/main/main.kicad_pcb (KiCad board)
At the start: 2 copper layers, 76.2 x 50.8 mm, 23 parts, among them J1 Molex2x15, J10 molex_01x02, J11 Conn_01x04, J12 Conn_01x08, J2 molex5P, J3 molex3P, J4 molex5P, J5 molex3P, J6 molex5P, J7 molex3P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

Commit message: v1.0
Other:
- board text removed: "WayWayWay"
Changed lines of the file:
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@@
 			(drillshape 0)
 			(scaleselection 1)
-			(outputdirectory "../gerbers for main pcb for standing frame v1.0/")
+			(outputdirectory "../../control/gerbers for control pcb for standing frame v1.0/")
 		)
 	)
@@
 		)
 	)
-	(gr_text "WayWayWay"
-		(at 118.237 72.644 0)
-		(layer "F.SilkS")
-		(effects
-			(font
-				(size 1.5 1.5)
-				(thickness 0.15)
-			)
-			(justify left bottom)
-		)
-	)
