File: main/main/main.kicad_pcb (KiCad board)
At the start: 2 copper layers, 76.2 x 50.8 mm, 23 parts, among them J1 Molex2x15, J10 molex_01x02, J11 Conn_01x04, J12 Conn_01x08, J2 molex5P, J3 molex3P, J4 molex5P, J5 molex3P, J6 molex5P, J7 molex3P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

Commit message: v1.4
Parts:
- removed G***: LOGO, LOGO
- moved BT1 6.96 mm to (173.5, 64.4), turned to 0 degrees
- moved TP1 4.55 mm to (173.5, 82.9), turned to 0 degrees
Connections:
- TP1 pad 1: Net-(U1-28_RX7) -> Net-(U1-24_A10_TX6_SCL2)
- U1 pad 16: Net-(J7-Pin_1) -> Net-(U1-24_A10_TX6_SCL2)
- U1 pad 20: Net-(U1-28_RX7) -> Net-(J7-Pin_1)
Routing:
- net Net-(U1-24_A10_TX6_SCL2): track 0.00 -> 25.8 mm
- net Net-(U1-28_RX7): track 16.6 -> 0.00 mm
- net Net-(J7-Pin_1): track 20.1 -> 27.3 mm
- net Net-(BT1-+): track 20.9 -> 23.0 mm
- net Net-(J1-Pin_15): track 39.1 -> 40.1 mm
- net GND: vias 0 -> 2
- added copper zone on B.Cu, net GND
Other:
- board text added: "+ bat - clock"
- board text added: "24"
- board text added: "v1.4"
- board text removed: "28"
- board text removed: "bat+"
- board text removed: "v1.0"
