File: main/main/main.kicad_sch (KiCad schematic)
At the start: 18 parts, among them J1 Molex2x15, J10 molex_01x02, J11 Conn_01x04, J12 Conn_01x08, J2 molex5P, J3 molex3P, J4 molex5P, J5 molex3P, J6 molex5P, J7 molex3P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

Commit message: v1.4
Connections:
- net GND: no longer U1.58 (GND), U1.59 (GND)
- net at U1.16 (24_A10_TX6_SCL2): now also TP1.1; no longer J7.1 (Pin_1)
- net at U1.20 (28_RX7): now also J7.1 (Pin_1); no longer TP1.1
- no-connect marks 14 -> 11
Changed lines of the file:
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@@
 	(title_block
 		(title "main PCB for standing frame")
-		(date "2024-07-10")
-		(rev "v1.0")
+		(date "2024-07-20")
+		(rev "v1.4")
 		(company "PNW Assistive Technology")
 		(comment 1 "Joshua Phelps")
@@
 	)
 	(junction
-		(at 106.68 120.65)
-		(diameter 0)
-		(color 0 0 0 0)
-	)
-	(junction
 		(at 134.62 134.62)
 		(diameter 0)
@@
 	)
 	(no_connect
-		(at 106.68 113.03)
-	)
-	(no_connect
 		(at 62.23 114.3)
 	)
 	(no_connect
-		(at 106.68 115.57)
-	)
-	(no_connect
-		(at 106.68 118.11)
-	)
-	(no_connect
 		(at 213.36 113.03)
 	)
@@
 	(wire
 		(pts
-			(xy 97.79 81.28) (xy 97.79 100.33)
-		)
-		(stroke
-			(width 0)
-			(type default)
-		)
-	)
-	(wire
-		(pts
 			(xy 52.07 102.87) (xy 52.07 109.22)
 		)
@@
 	(wire
 		(pts
+			(xy 100.33 99.06) (xy 100.33 91.44)
+		)
+		(stroke
+			(width 0)
+			(type default)
+		)
+	)
+	(wire
+		(pts
 			(xy 162.56 43.18) (xy 175.26 43.18)
 		)
@@
 	(wire
 		(pts
+			(xy 101.6 81.28) (xy 101.6 96.52)
+		)
+		(stroke
+			(width 0)
+			(type default)
+		)
+	)
+	(wire
+		(pts
 			(xy 195.58 60.96) (xy 195.58 55.88)
 		)
@@
 	(wire
 		(pts
+			(xy 101.6 81.28) (xy 106.68 81.28)
+		)
+		(stroke
+			(width 0)
+			(type default)
+		)
+	)
+	(wire
+		(pts
 			(xy 134.62 134.62) (xy 134.62 140.97)
 		)
@@
 	(wire
 		(pts
-			(xy 106.68 120.65) (xy 106.68 123.19)
-		)
-		(stroke
-			(width 0)
-			(type default)
-		)
-	)
-	(wire
-		(pts
 			(xy 104.14 96.52) (xy 106.68 96.52)
 		)
@@
 	(wire
 		(pts
+			(xy 43.18 90.17) (xy 49.53 90.17)
+		)
+		(stroke
+			(width 0)
+			(type default)
+		)
+	)
+	(wire
+		(pts
 			(xy 236.22 62.23) (xy 236.22 63.5)
 		)
@@
 	(wire
 		(pts
-			(xy 162.56 96.52) (xy 165.1 96.52)
+			(xy 49.53 99.06) (xy 100.33 99.06)
 		)
 		(stroke
@@
 	(wire
 		(pts
-			(xy 130.81 67.31) (xy 106.68 67.31)
+			(xy 162.56 96.52) (xy 165.1 96.52)
 		)
 		(stroke
@@
 	(wire
 		(pts
-			(xy 236.22 80.01) (xy 203.2 80.01)
+			(xy 130.81 67.31) (xy 106.68 67.31)
 		)
 		(stroke
@@
 	(wire
 		(pts
-			(xy 91.44 80.01) (xy 49.53 80.01)
+			(xy 236.22 80.01) (xy 203.2 80.01)
 		)
 		(stroke
@@
 	(wire
 		(pts
-			(xy 236.22 78.74) (xy 236.22 77.47)
+			(xy 91.44 80.01) (xy 49.53 80.01)
 		)
 		(stroke
@@
 	(wire
 		(pts
-			(xy 165.1 97.79) (xy 219.71 97.79)
+			(xy 236.22 78.74) (xy 236.22 77.47)
 		)
 		(stroke
@@
 	(wire
 		(pts
-			(xy 171.45 91.44) (xy 162.56 91.44)
+			(xy 165.1 97.79) (xy 219.71 97.79)
 		)
 		(stroke
@@
 	(wire
 		(pts
-			(xy 43.18 72.39) (xy 48.26 72.39)
+			(xy 171.45 91.44) (xy 162.56 91.44)
 		)
 		(stroke
@@
 	(wire
 		(pts
-			(xy 49.53 90.17) (xy 43.18 90.17)
+			(xy 43.18 72.39) (xy 48.26 72.39)
 		)
 		(stroke
@@
 	(wire
 		(pts
-			(xy 49.53 100.33) (xy 49.53 90.17)
-		)
-		(stroke
-			(width 0)
-			(type default)
-		)
-	)
-	(wire
-		(pts
 			(xy 162.56 86.36) (xy 173.99 86.36)
 		)
@@
 	(wire
 		(pts
-			(xy 104.14 120.65) (xy 106.68 120.65)
-		)
-		(stroke
-			(width 0)
-			(type default)
-		)
-	)
-	(wire
-		(pts
 			(xy 195.58 55.88) (xy 162.56 55.88)
 		)
@@
 	(wire
 		(pts
+			(xy 100.33 91.44) (xy 106.68 91.44)
+		)
+		(stroke
+			(width 0)
+			(type default)
+		)
+	)
+	(wire
+		(pts
 			(xy 205.74 113.03) (xy 205.74 74.93)
 		)
@@
 	(wire
 		(pts
+			(xy 49.53 90.17) (xy 49.53 99.06)
+		)
+		(stroke
+			(width 0)
+			(type default)
+		)
+	)
+	(wire
+		(pts
 			(xy 62.23 92.71) (xy 96.52 92.71)
 		)
@@
 	(wire
 		(pts
-			(xy 97.79 100.33) (xy 49.53 100.33)
-		)
-		(stroke
-			(width 0)
-			(type default)
-		)
-	)
-	(wire
-		(pts
 			(xy 162.56 68.58) (xy 168.91 68.58)
 		)
@@
 	(wire
 		(pts
-			(xy 101.6 91.44) (xy 106.68 91.44)
-		)
-		(stroke
-			(width 0)
-			(type default)
-		)
-	)
-	(wire
-		(pts
 			(xy 134.62 130.81) (xy 134.62 134.62)
 		)
@@
 	(wire
 		(pts
-			(xy 97.79 81.28) (xy 106.68 81.28)
-		)
-		(stroke
-			(width 0)
-			(type default)
-		)
-	)
-	(wire
-		(pts
 			(xy 92.71 81.28) (xy 92.71 58.42)
 		)
@@
 	(wire
 		(pts
-			(xy 101.6 96.52) (xy 101.6 91.44)
-		)
-		(stroke
-			(width 0)
-			(type default)
-		)
-	)
-	(wire
-		(pts
 			(xy 83.82 53.34) (xy 83.82 46.99)
 		)
@@
 		(pin "50"
 		)
-		(pin "56"
-		)
-		(pin "55"
-		)
 		(pin "51"
 		)
-		(pin "59"
-		)
 		(pin "3"
 		)
@@
 		(pin "46"
 		)
-		(pin "49"
-		)
-		(pin "58"
-		)
 		(pin "48"
 		)
@@
 		(pin "45"
 		)
-		(pin "57"
-		)
 		(instances
 			(project ""
@@
 	(symbol
 		(lib_id "power:GND")
-		(at 104.14 120.65 0)
-		(unit 1)
-		(exclude_from_sim no)
-		(in_bom yes)
-		(on_board yes)
-		(dnp no)
-		(property "Reference" "#PWR019"
-			(at 104.14 127 0)
-			(effects
-				(font
-					(size 1.27 1.27)
-				)
-				(hide yes)
-			)
-		)
-		(property "Value" "GND"
-			(at 101.6 121.158 0)
-			(effects
-				(font
-					(size 1.27 1.27)
-				)
-			)
-		)
-		(property "Footprint" ""
-			(at 104.14 120.65 0)
-			(effects
-				(font
-					(size 1.27 1.27)
-				)
-				(hide yes)
-			)
-		)
-		(property "Datasheet" ""
-			(at 104.14 120.65 0)
-			(effects
-				(font
-					(size 1.27 1.27)
-				)
-				(hide yes)
-			)
-		)
-		(property "Description" "Power symbol creates a global label with name \"GND\" , ground"
-			(at 104.14 120.65 0)
-			(effects
-				(font
-					(size 1.27 1.27)
-				)
-				(hide yes)
-			)
-		)
-		(pin "1"
-		)
-		(instances
-			(project "main"
-				(path "/ab47a88c-4e7b-4d2a-8992-259f4c293a97"
-					(reference "#PWR019")
-					(unit 1)
-				)
-			)
-		)
-	)
-	(symbol
-		(lib_id "power:GND")
 		(at 62.23 77.47 0)
 		(unit 1)
@@
 		(dnp no)
 		(property "Reference" "J12"
-			(at 191.262 113.03 0)
+			(at 195.072 118.618 90)
 			(effects
 				(font
@@
 		)
 		(property "Value" "Conn_01x08"
-			(at 193.802 113.03 0)
+			(at 211.582 118.11 90)
 			(effects
 				(font
