File: control/control/control.kicad_pcb (KiCad board)
At the start: 2 copper layers, 76.2 x 101.6 mm, 34 parts, among them J1 Molex2x15, Q1 2N3904, Q2 2N3904, Q3 2N3904, SW3 221ADC16, SW4 221ADC16, SW5 221ADC16, SW6 221ADC16, SW7 221ADC16, U1 LM3914N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

Commit message: v1.0
Other:
- board text removed: "WayWayWay"
Changed lines of the file:
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@@
-		)
-	)
-	(gr_text "WayWayWay"
-		(at 111.252 67.056 0)
-		(layer "F.SilkS")
-		(effects
-			(font
-				(size 1 1)
-				(thickness 0.15)
-			)
-			(justify left bottom)
 		)
 	)

Commit message: v1.4
Parts:
- removed G***: LOGO, LOGO
- added NT1: NetTie_2, Jumper:SolderJumper-2_P1.3mm_Bridged_RoundedPad1.0x1.5mm, F.Cu at (149.7, 53.0)
- added R14: 0, Resistor_THT:R_Axial_DIN0207_L6.3mm_D2.5mm_P10.16mm_Horizontal, F.Cu at (154.8, 53.0)
- moved SW1 9.30 mm to (149.3, 132.5)
Connections:
- S1 pad L1: 3.3V -> Net-(S1-A)
Routing:
- net 3.3V: track 263.8 -> 225.3 mm
- net Net-(S1-A): track 0.00 -> 35.4 mm
- net GND: vias 4 -> 6
Other:
- board text added: "- +"
- board text added: "v1.4"

Commit message: update control v1.4
Parts:
- moved REF** 1.91 mm to (105.4, 146.7)
- moved REF** 1.91 mm to (174.0, 146.7)
- moved BAR1 0.63 mm to (110.6, 121.9)
Routing:
- net Net-(J1-Pin_26): track 167.4 -> 150.7 mm
- net 3.3V: track 225.3 -> 224.2 mm
- net Net-(U1-LED9): track 3.70 -> 3.07 mm
- net Net-(U1-LED8): track 3.70 -> 3.07 mm
- net Net-(U1-LED7): track 3.70 -> 3.07 mm
- net Net-(U1-LED6): track 3.70 -> 3.07 mm
- net Net-(U1-LED5): track 3.70 -> 3.07 mm
- net Net-(U1-LED4): track 3.70 -> 3.07 mm
- net Net-(U1-LED3): track 3.70 -> 3.07 mm
- net Net-(U1-LED2): track 3.70 -> 3.07 mm
- net Net-(U1-LED10): track 3.70 -> 3.07 mm
- net Net-(U1-LED1): track 12.4 -> 11.7 mm
Other:
- board size 76.2 x 101.6 mm -> 76.2 x 99.7 mm
